File: WD1M_RFM9x.brd (EAGLE design)
At the start: 25.4 x 33 mm, 17 parts, among them U2 MICROCHIP-24AA02E64T_24AA02E6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

Commit message: Work halted, Minor updates before archiving
Parts:
- R1, R2: value 4.7k -> 2k
Changed lines of the file:
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@@
 </element>
 <element name="U$2" library="diy-modules" package="WIRELESS-LORA-RFM95W#SMD" value="WIRELESS-LORA-RFM95W#SMD" x="12.7" y="16.51" rot="MR270"/>
-<element name="R1" library="rcl" package="R0805" value="4.7k" x="30.48" y="5.334"/>
-<element name="R2" library="rcl" package="R0805" value="4.7k" x="30.48" y="2.032"/>
+<element name="R1" library="rcl" package="R0805" value="2k" x="30.48" y="5.334"/>
+<element name="R2" library="rcl" package="R0805" value="2k" x="30.48" y="2.032"/>
 <element name="C2" library="rcl" package="C0805K" value="100n" x="29.972" y="14.224" rot="R180"/>
 <element name="C3" library="rcl" package="C0805K" value="100n" x="37.338" y="6.604" rot="R180"/>

Commit message: FIT/NOFIT change
Parts:
- D2: value (none) -> NOFIT
Changed lines of the file:
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@@
 <element name="D3" library="adafruit" package="SOD-323F" value="" x="9.906" y="9.906" rot="R90"/>
 <element name="D1" library="adafruit" package="SOD-323F" value="" x="7.874" y="9.906" rot="R90"/>
-<element name="D2" library="adafruit" package="SOD-323F" value="" x="5.842" y="9.906" rot="R90"/>
+<element name="D2" library="adafruit" package="SOD-323F" value="NOFIT" x="5.842" y="9.906" rot="R90"/>
 <element name="D4" library="SparkFun-LED" package="WS2812B" value="" x="7.62" y="22.86" rot="R90"/>
 <element name="D5" library="SparkFun-LED" package="WS2812B" value="" x="18.034" y="22.86" rot="R90"/>
