File: WD1M_RFM9x.sch (EAGLE design)
At the start: 17 parts, among them U2 MICROCHIP-24AA02E64T_24AA02E6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

Commit message: Work halted, Minor updates before archiving
Parts:
- R1, R2: value 4.7k -> 2k
Changed lines of the file:
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@@
 <part name="P+7" library="freetronics-original" deviceset="3.3V" device=""/>
 <part name="GND7" library="freetronics-original" deviceset="GND" device=""/>
-<part name="R1" library="rcl" deviceset="R-EU_" device="R0805" value="4.7k"/>
-<part name="R2" library="rcl" deviceset="R-EU_" device="R0805" value="4.7k"/>
+<part name="R1" library="rcl" deviceset="R-EU_" device="R0805" value="2k"/>
+<part name="R2" library="rcl" deviceset="R-EU_" device="R0805" value="2k"/>
 <part name="C2" library="rcl" deviceset="C-EU" device="C0805K" value="100n"/>
 <part name="C3" library="rcl" deviceset="C-EU" device="C0805K" value="100n"/>

Commit message: FIT/NOFIT change
Parts:
- D2: value (none) -> NOFIT
Other:
- note added: "D2 MAY NEED TO BE NO FIT DUE TO DIO2 BEING HIGH AT BOOTUP."
Changed lines of the file:
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@@
 <part name="D3" library="adafruit" deviceset="DIODE" device="SOD-323F"/>
 <part name="D1" library="adafruit" deviceset="DIODE" device="SOD-323F"/>
-<part name="D2" library="adafruit" deviceset="DIODE" device="SOD-323F"/>
+<part name="D2" library="adafruit" deviceset="DIODE" device="SOD-323F" value="NOFIT"/>
 <part name="D4" library="SparkFun-LED" deviceset="WS2812B" device=""/>
 <part name="D5" library="SparkFun-LED" deviceset="WS2812B" device=""/>
@@
 <text x="101.6" y="71.12" size="1.778" layer="91">RST active low same as ESP8266</text>
 <text x="25.4" y="170.18" size="1.778" layer="91">USING 0805 FOR EASE OF SELF BUILD</text>
+<text x="119.38" y="55.88" size="1.778" layer="91">D2 MAY NEED TO BE NO FIT
+DUE TO DIO2 BEING HIGH
+AT BOOTUP.</text>
 </plain>
 <instances>
